File: schematic/lightmeter_proto3.brd (EAGLE design)
At the start: 28 x 51.9 mm, 75 parts, among them J1 AVR_SPI_PRG_6NS, Q1 NCHANNELMOSFET, Q10 NCHANNELMOSFET, Q11 NCHANNELMOSFET, Q12 NCHANNELMOSFET, Q16 PCHANNELMOSFET, Q2 PCHANNELMOSFET, Q3 NCHANNELMOSFET, Q4 PCHANNELMOSFET, Q5 NCHANNELMOSFET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

Commit message: Make naming of values systematic in proto boards.
Parts:
- C10, C11: value 1µ -> 1u
- C12, C6, C7, C8, C9: value 4µ7 -> 4u7
- C14, C16: value µ1 -> u1
- C18, C2, L2: value 2µ2 -> 2u2
- R1, R2: value 15K -> 15k
- R16, R18: value 10K% -> 10k
- R17, R25: value 10K -> 10k
- R19: value 6K8% -> 6k8%
- R21: value 16K -> 16k
- R3, R4: value 1K -> 1k
Changed lines of the file:
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@@
 </autorouter>
 <elements>
-<element name="C16" library="rcl" package="C0402" value="µ1" x="6.35" y="35.687"/>
+<element name="C16" library="rcl" package="C0402" value="u1" x="6.35" y="35.687"/>
 <element name="C15" library="rcl" package="C0402" value="4u7" x="15.494" y="26.67"/>
-<element name="C11" library="rcl" package="C0402" value="1µ" x="17.018" y="45.847" smashed="yes">
+<element name="C11" library="rcl" package="C0402" value="1u" x="17.018" y="45.847" smashed="yes">
 <attribute name="NAME" x="16.643559375" y="46.369059375" size="1.27" layer="25"/>
 <attribute name="VALUE" x="16.383003125" y="43.942" size="1.27" layer="27"/>
 </element>
-<element name="C9" library="rcl" package="C0402" value="4µ7" x="20.32" y="33.655"/>
-<element name="C8" library="rcl" package="C0402" value="4µ7" x="20.32" y="37.465"/>
-<element name="C7" library="rcl" package="C0402" value="4µ7" x="20.32" y="41.402"/>
-<element name="C6" library="rcl" package="C0402" value="4µ7" x="20.32" y="45.085"/>
+<element name="C9" library="rcl" package="C0402" value="4u7" x="20.32" y="33.655"/>
+<element name="C8" library="rcl" package="C0402" value="4u7" x="20.32" y="37.465"/>
+<element name="C7" library="rcl" package="C0402" value="4u7" x="20.32" y="41.402"/>
+<element name="C6" library="rcl" package="C0402" value="4u7" x="20.32" y="45.085"/>
 <element name="C1" library="rcl" package="C0402" value="4u7" x="10.287" y="25.527" rot="R90"/>
-<element name="C14" library="rcl" package="C0402" value="µ1" x="17.653" y="49.022" rot="R270"/>
-<element name="C10" library="rcl" package="C0402" value="1µ" x="22.606" y="42.926" rot="R90"/>
-<element name="C12" library="rcl" package="C0402" value="4µ7" x="24.384" y="48.895" rot="R30"/>
+<element name="C14" library="rcl" package="C0402" value="u1" x="17.653" y="49.022" rot="R270"/>
+<element name="C10" library="rcl" package="C0402" value="1u" x="22.606" y="42.926" rot="R90"/>
+<element name="C12" library="rcl" package="C0402" value="4u7" x="24.384" y="48.895" rot="R30"/>
 <element name="D10" library="lightmeter" package="VEMD2523SLX01" value="VEMD2523SLX01" x="22.352" y="47.752" smashed="yes">
 <attribute name="NAME" x="18.542" y="52.324" size="1.27" layer="26"/>
@@
 <attribute name="PROD_ID" value="CONN-08352" x="5.08" y="17.272" size="1.778" layer="27" rot="R270" display="off"/>
 </element>
-<element name="L2" library="microbuilder" package="_0603" value="2µ2" x="12.7" y="26.67"/>
+<element name="L2" library="microbuilder" package="_0603" value="2u2" x="12.7" y="26.67"/>
 <element name="Q1" library="lightmeter" package="SOT-416-3" value="NCHANNELMOSFET" x="24.13" y="43.18"/>
 <element name="Q8" library="lightmeter" package="SOT-416-3" value="NCHANNELMOSFET" x="2.413" y="46.482"/>
@@
 </element>
 <element name="Q7" library="lightmeter" package="SOT-416-3" value="PCHANNELMOSFET" x="14.732" y="36.576"/>
-<element name="R17" library="resistor" package="R0402" value="10K" x="22.4282" y="29.845" smashed="yes" rot="R270">
+<element name="R17" library="resistor" package="R0402" value="10k" x="22.4282" y="29.845" smashed="yes" rot="R270">
 <attribute name="SPICEPREFIX" value="R" x="22.4282" y="29.845" size="1.778" layer="27" rot="R270" display="off"/>
 <attribute name="NAME" x="22.1742" y="29.083" size="1.27" layer="25" rot="R270"/>
@@
 <attribute name="SPICEPREFIX" value="R" x="6.8072" y="43.1038" size="1.778" layer="27" display="off"/>
 </element>
-<element name="R21" library="resistor" package="R0402" value="16K" x="18.796" y="6.985" rot="R90">
+<element name="R21" library="resistor" package="R0402" value="16k" x="18.796" y="6.985" rot="R90">
 <attribute name="SPICEPREFIX" value="R" x="18.796" y="6.985" size="1.778" layer="27" rot="R90" display="off"/>
 </element>
-<element name="R16" library="resistor" package="R0402" value="10K%" x="25.146" y="29.591" smashed="yes" rot="R90">
+<element name="R16" library="resistor" package="R0402" value="10k" x="25.146" y="29.591" smashed="yes" rot="R90">
 <attribute name="SPICEPREFIX" value="R" x="25.146" y="29.591" size="1.778" layer="27" rot="R90" display="off"/>
 <attribute name="NAME" x="22.606" y="32.131" size="1.27" layer="25"/>
@@
 <attribute name="VALUE" x="15.63" y="54.947" size="0.4064" layer="27" ratio="10" rot="R180"/>
 </element>
-<element name="R18" library="resistor" package="R0402" value="10K%" x="2.54" y="27.559">
+<element name="R18" library="resistor" package="R0402" value="10k" x="2.54" y="27.559">
 <attribute name="SPICEPREFIX" value="R" x="2.54" y="27.559" size="1.778" layer="27" display="off"/>
 </element>
-<element name="R19" library="resistor" package="R0402" value="6K8%" x="0.381" y="36.957" smashed="yes" rot="R90">
+<element name="R19" library="resistor" package="R0402" value="6k8%" x="0.381" y="36.957" smashed="yes" rot="R90">
 <attribute name="SPICEPREFIX" value="R" x="0.381" y="36.957" size="1.778" layer="27" rot="R90" display="off"/>
 <attribute name="NAME" x="2.287940625" y="35.485734375" size="1.27" layer="25" rot="R90"/>
 <attribute name="VALUE" x="2.413" y="36.321996875" size="1.27" layer="27" rot="R90"/>
 </element>
-<element name="R1" library="resistor" package="R0402" value="15K" x="19.685" y="21.209" smashed="yes" rot="R80">
+<element name="R1" library="resistor" package="R0402" value="15k" x="19.685" y="21.209" smashed="yes" rot="R80">
 <attribute name="SPICEPREFIX" value="R" x="19.685" y="21.209" size="1.778" layer="27" rot="R80" display="off"/>
 <attribute name="NAME" x="21.491309375" y="19.318965625" size="1.27" layer="25" rot="R80"/>
 <attribute name="VALUE" x="21.5758625" y="20.23079375" size="1.27" layer="27" rot="R80"/>
 </element>
-<element name="R2" library="resistor" package="R0402" value="15K" x="16.256" y="14.478" smashed="yes">
+<element name="R2" library="resistor" package="R0402" value="15k" x="16.256" y="14.478" smashed="yes">
 <attribute name="SPICEPREFIX" value="R" x="16.256" y="14.478" size="1.778" layer="27" display="off"/>
 <attribute name="NAME" x="14.605" y="12.446" size="1.27" layer="25"/>
@@
 </element>
 <element name="C17" library="rcl" package="C0402" value="4u7" x="17.399" y="10.16" rot="R90"/>
-<element name="R25" library="resistor" package="R0402" value="10K" x="8.382" y="27.432" rot="R90">
+<element name="R25" library="resistor" package="R0402" value="10k" x="8.382" y="27.432" rot="R90">
 <attribute name="SPICEPREFIX" value="R" x="8.382" y="27.432" size="1.778" layer="27" rot="R90" display="off"/>
 </element>
 <element name="Q16" library="lightmeter" package="SOT-416-3" value="PCHANNELMOSFET" x="6.604" y="29.718"/>
 <element name="D$1" library="lightmeter" package="SOT23" value="GSOT04-E3-08" x="13.589" y="11.303"/>
-<element name="C18" library="rcl" package="C0402" value="2µ2" x="6.223" y="49.911"/>
+<element name="C18" library="rcl" package="C0402" value="2u2" x="6.223" y="49.911"/>
 <element name="D1" library="diode2" package="SOD323-W" value="" x="13.716" y="15.875" rot="R270"/>
 <element name="D2" library="diode2" package="SOD323-W" value="" x="16.891" y="23.495" rot="R90"/>
-<element name="C2" library="rcl" package="C0402" value="2µ2" x="7.874" y="44.958" rot="R180"/>
+<element name="C2" library="rcl" package="C0402" value="2u2" x="7.874" y="44.958" rot="R180"/>
 <element name="IC$6" library="lightmeter" package="DFN-10" value="MMA8653" x="2.667" y="32.004" rot="R270"/>
 <element name="C3" library="rcl" package="C0402" value="1u" x="3.175" y="30.099"/>
@@
 <attribute name="VALUE" x="2.286" y="31.877" size="1.27" layer="27" rot="R90"/>
 </element>
-<element name="R3" library="resistor" package="R0402" value="1K" x="0.254" y="29.4894" smashed="yes" rot="R90">
+<element name="R3" library="resistor" package="R0402" value="1k" x="0.254" y="29.4894" smashed="yes" rot="R90">
 <attribute name="SPICEPREFIX" value="R" x="0.254" y="29.4894" size="1.778" layer="27" rot="R90" display="off"/>
 <attribute name="NAME" x="2.032" y="28.8544" size="1.27" layer="25" rot="R90"/>
 <attribute name="VALUE" x="2.286" y="28.8544" size="1.27" layer="27" rot="R90"/>
 </element>
-<element name="R4" library="resistor" package="R0402" value="1K" x="3.683" y="34.5186">
+<element name="R4" library="resistor" package="R0402" value="1k" x="3.683" y="34.5186">
 <attribute name="SPICEPREFIX" value="R" x="3.683" y="34.5186" size="1.778" layer="27" display="off"/>
 </element>
