File: schematic/lightmeter.sch (EAGLE design)
At the start: 77 parts, among them J1 CONNECTEDJUMPER, J2 CONNECTEDJUMPER, J3 CONNECTEDJUMPER, J4 CONNECTEDJUMPER, J5 CONNECTEDJUMPER, J6 CONNECTEDJUMPER, Q1 PCHANNELMOSFETSOT-523-3-BTTM

Commit message: More work on board/schematic.
Parts:
- R7: value 10k -> 390k
Connections:
- removed net FLASHSYNC: IC$4.PB1
- net NRST: no longer U1.USBID
- net VCC: no longer R1.1
- net VUSB: now also R1.1
Changed lines of the file:
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@@
 <part name="C17" library="rcl" deviceset="C-EU" device="C0402" value="u1"/>
 <part name="GND15" library="supply1" deviceset="GND" device=""/>
-<part name="R7" library="resistor" deviceset="R-EU_" device="R0402" value="10k"/>
+<part name="R7" library="resistor" deviceset="R-EU_" device="R0402" value="390k"/>
 <part name="GND8" library="supply1" deviceset="GND" device=""/>
 <part name="R10" library="resistor" deviceset="R-EU_" device="R0402" value="390k"/>
@@
 <part name="Q2" library="microbuilder" deviceset="MOSFET-P" device="WIDE"/>
 <part name="Q3" library="microbuilder" deviceset="MOSFET-P" device="WIDE"/>
-<part name="P+5" library="supply1" deviceset="VCC" device=""/>
 <part name="D4" library="adafruit" deviceset="DIODE" device="SOD-323F"/>
 <part name="D1" library="lightmeter" deviceset="SCHOTTKY-DIODE" device="SOD-929"/>
@@
 <instance part="Q2" gate="G$1" x="86.36" y="-35.56" rot="R270"/>
 <instance part="Q3" gate="G$1" x="119.38" y="-35.56" rot="R270"/>
-<instance part="P+5" gate="VCC" x="-122.936" y="60.96" rot="R90"/>
 <instance part="D4" gate="G$1" x="-15.24" y="-86.36"/>
 <instance part="D1" gate="G$1" x="96.52" y="40.64" rot="R90"/>
@@
 <wire x1="-121.92" y1="-124.46" x2="-116.84" y2="-124.46" width="0.1524" layer="91"/>
 </segment>
-<segment>
-<pinref part="R1" gate="G$1" pin="1"/>
-<pinref part="P+5" gate="VCC" pin="VCC"/>
-<wire x1="-120.396" y1="60.96" x2="-116.078" y2="60.96" width="0.1524" layer="91"/>
-</segment>
 </net>
 <net name="VREG" class="0">
@@
 <wire x1="0" y1="-22.86" x2="2.54" y2="-22.86" width="0.1524" layer="91"/>
 <label x="2.54" y="-22.86" size="1.778" layer="95" xref="yes"/>
-</segment>
-</net>
-<net name="FLASHSYNC" class="0">
-<segment>
-<pinref part="IC$4" gate="G$1" pin="PB1"/>
-<wire x1="-20.32" y1="-43.18" x2="-20.32" y2="-45.72" width="0.1524" layer="91"/>
-<label x="-20.32" y="-45.72" size="1.778" layer="95" rot="R270" xref="yes"/>
 </segment>
 </net>
@@
 <wire x1="-132.08" y1="-38.1" x2="-137.16" y2="-38.1" width="0.1524" layer="91"/>
 <label x="-139.7" y="-48.26" size="1.778" layer="95" rot="R180" xref="yes"/>
+</segment>
+<segment>
+<pinref part="R1" gate="G$1" pin="1"/>
+<wire x1="-120.396" y1="60.96" x2="-116.078" y2="60.96" width="0.1524" layer="91"/>
+<label x="-119.38" y="60.96" size="1.778" layer="95" rot="R180" xref="yes"/>
 </segment>
 </net>
@@
 <pinref part="R5" gate="G$1" pin="1"/>
 </segment>
-<segment>
-<pinref part="U1" gate="G$1" pin="USBID"/>
-<wire x1="-83.82" y1="66.04" x2="-85.09" y2="66.04" width="0.1524" layer="91"/>
-<label x="-85.09" y="66.04" size="1.778" layer="95" rot="R180" xref="yes"/>
-</segment>
-</net>
+</net>

Commit message: More work on board/schematic.
Parts:
- added RST: TPB1,27, testpad:TPB1,27
Connections:
- net NRST: now also RST.TP
Changed lines of the file:
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@@
 <part name="Q1" library="lightmeter" deviceset="PCHANNELMOSFET" device="SOT-523-3-BTTM" value="PCHANNELMOSFETSOT-523-3-BTTM"/>
 <part name="D5" library="adafruit" deviceset="DIODE" device="SOD-323F"/>
+<part name="RST" library="testpad" deviceset="TP" device="B1,27"/>
 </parts>
 <sheets>
@@
 <instance part="Q1" gate="G$1" x="157.48" y="15.24" rot="R90"/>
 <instance part="D5" gate="G$1" x="0" y="-86.36" rot="R180"/>
+<instance part="RST" gate="G$1" x="-109.22" y="-2.54" rot="R90"/>
 </instances>
 <busses>
@@
 <label x="-101.6" y="-7.62" size="1.778" layer="95" rot="R180" xref="yes"/>
 <wire x1="-99.06" y1="-7.62" x2="-101.6" y2="-7.62" width="0.1524" layer="91"/>
-<wire x1="-99.06" y1="-7.62" x2="-99.06" y2="2.54" width="0.1524" layer="91"/>
+<wire x1="-99.06" y1="-7.62" x2="-99.06" y2="-2.54" width="0.1524" layer="91"/>
 <junction x="-99.06" y="-7.62"/>
 <pinref part="R5" gate="G$1" pin="1"/>
-</segment>
-</net>
+<pinref part="RST" gate="G$1" pin="TP"/>
+<wire x1="-99.06" y1="-2.54" x2="-99.06" y2="2.54" width="0.1524" layer="91"/>
+<wire x1="-99.06" y1="-2.54" x2="-106.68" y2="-2.54" width="0.1524" layer="91"/>
+<junction x="-99.06" y="-2.54"/>
+</segment>
+</net>
