File: schematic/lightmeter.sch (EAGLE design)
At the start: 91 parts, among them J1 CONNECTEDJUMPER, J2 CONNECTEDJUMPER, J3 CONNECTEDJUMPER, J4 CONNECTEDJUMPER, J5 CONNECTEDJUMPER, J6 CONNECTEDJUMPER, J7 CONNECTEDJUMPER, Q1 PCHANNELMOSFETSOT-523-3-BTTM, Y1 8MHz

Commit message: Some progress on metering mess.
Parts:
- R11: value 10k (0.1%) -> 500 (0.1%)
- R12: value 10k (0.1% -> 500 (0.1%
Changed lines of the file:
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@@
 <part name="C23" library="rcl" deviceset="C-EU" device="C0402" value="u1"/>
 <part name="C31" library="rcl" deviceset="C-EU" device="C0402" value="u1"/>
-<part name="R11" library="resistor" deviceset="R-EU_" device="R0402" value="10k (0.1%)"/>
+<part name="R11" library="resistor" deviceset="R-EU_" device="R0402" value="500 (0.1%)"/>
 <part name="R14" library="resistor" deviceset="R-EU_" device="R0402" value="10k"/>
-<part name="R12" library="resistor" deviceset="R-EU_" device="R0402" value="10k (0.1%"/>
+<part name="R12" library="resistor" deviceset="R-EU_" device="R0402" value="500 (0.1%"/>
 <part name="D6" library="adafruit" deviceset="DIODE" device="SOD-323F"/>
 <part name="D1" library="lightmeter" deviceset="SCHOTTKY-DIODE" device="SOD-923-BTTM"/>

Commit message: Is it finally fixed (??)
Parts:
- R12: value 500 (0.1% -> 500 (0.1%)
Changed lines of the file:
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@@
 <part name="R11" library="resistor" deviceset="R-EU_" device="R0402" value="500 (0.1%)"/>
 <part name="R14" library="resistor" deviceset="R-EU_" device="R0402" value="10k"/>
-<part name="R12" library="resistor" deviceset="R-EU_" device="R0402" value="500 (0.1%"/>
+<part name="R12" library="resistor" deviceset="R-EU_" device="R0402" value="500 (0.1%)"/>
 <part name="D6" library="adafruit" deviceset="DIODE" device="SOD-323F"/>
 <part name="D1" library="lightmeter" deviceset="SCHOTTKY-DIODE" device="SOD-923-BTTM"/>

Commit message: Some improvements to ground plane connectivity.
Connections:
- net BATVOLTAGE: now also IC$4.PB5; no longer IC$4.PB0
Changed lines of the file:
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@@
 <grid distance="0.1" unitdist="inch" unit="inch" style="lines" multiple="1" display="no" altdistance="0.01" altunitdist="inch" altunit="inch"/>
 <layers>
-<layer number="1" name="Top" color="4" fill="1" visible="no" active="no"/>
-<layer number="2" name="Route2" color="1" fill="3" visible="no" active="no"/>
-<layer number="3" name="Route3" color="4" fill="3" visible="no" active="no"/>
-<layer number="4" name="Route4" color="1" fill="4" visible="no" active="no"/>
-<layer number="5" name="Route5" color="4" fill="4" visible="no" active="no"/>
-<layer number="6" name="Route6" color="1" fill="8" visible="no" active="no"/>
-<layer number="7" name="Route7" color="4" fill="8" visible="no" active="no"/>
-<layer number="8" name="Route8" color="1" fill="2" visible="no" active="no"/>
-<layer number="9" name="Route9" color="4" fill="2" visible="no" active="no"/>
-<layer number="10" name="Route10" color="1" fill="7" visible="no" active="no"/>
-<layer number="11" name="Route11" color="4" fill="7" visible="no" active="no"/>
-<layer number="12" name="Route12" color="1" fill="5" visible="no" active="no"/>
-<layer number="13" name="Route13" color="4" fill="5" visible="no" active="no"/>
-<layer number="14" name="Route14" color="1" fill="6" visible="no" active="no"/>
-<layer number="15" name="Route15" color="4" fill="6" visible="no" active="no"/>
-<layer number="16" name="Bottom" color="1" fill="1" visible="no" active="no"/>
-<layer number="17" name="Pads" color="2" fill="1" visible="no" active="no"/>
-<layer number="18" name="Vias" color="2" fill="1" visible="no" active="no"/>
-<layer number="19" name="Unrouted" color="6" fill="1" visible="no" active="no"/>
-<layer number="20" name="Dimension" color="15" fill="1" visible="no" active="no"/>
-<layer number="21" name="tPlace" color="7" fill="1" visible="no" active="no"/>
-<layer number="22" name="bPlace" color="7" fill="1" visible="no" active="no"/>
-<layer number="23" name="tOrigins" color="15" fill="1" visible="no" active="no"/>
-<layer number="24" name="bOrigins" color="15" fill="1" visible="no" active="no"/>
-<layer number="25" name="tNames" color="7" fill="1" visible="no" active="no"/>
-<layer number="26" name="bNames" color="7" fill="1" visible="no" active="no"/>
-<layer number="27" name="tValues" color="7" fill="1" visible="no" active="no"/>
-<layer number="28" name="bValues" color="7" fill="1" visible="no" active="no"/>
+<layer number="1" name="Top" color="4" fill="1" visible="yes" active="no"/>
+<layer number="2" name="Route2" color="1" fill="3" visible="yes" active="no"/>
+<layer number="3" name="Route3" color="4" fill="3" visible="yes" active="no"/>
+<layer number="4" name="Route4" color="1" fill="4" visible="yes" active="no"/>
+<layer number="5" name="Route5" color="4" fill="4" visible="yes" active="no"/>
+<layer number="6" name="Route6" color="1" fill="8" visible="yes" active="no"/>
+<layer number="7" name="Route7" color="4" fill="8" visible="yes" active="no"/>
+<layer number="8" name="Route8" color="1" fill="2" visible="yes" active="no"/>
+<layer number="9" name="Route9" color="4" fill="2" visible="yes" active="no"/>
+<layer number="10" name="Route10" color="1" fill="7" visible="yes" active="no"/>
+<layer number="11" name="Route11" color="4" fill="7" visible="yes" active="no"/>
+<layer number="12" name="Route12" color="1" fill="5" visible="yes" active="no"/>
+<layer number="13" name="Route13" color="4" fill="5" visible="yes" active="no"/>
+<layer number="14" name="Route14" color="1" fill="6" visible="yes" active="no"/>
+<layer number="15" name="Route15" color="4" fill="6" visible="yes" active="no"/>
+<layer number="16" name="Bottom" color="1" fill="1" visible="yes" active="no"/>
+<layer number="17" name="Pads" color="2" fill="1" visible="yes" active="no"/>
+<layer number="18" name="Vias" color="2" fill="1" visible="yes" active="no"/>
+<layer number="19" name="Unrouted" color="6" fill="1" visible="yes" active="no"/>
+<layer number="20" name="Dimension" color="15" fill="1" visible="yes" active="no"/>
+<layer number="21" name="tPlace" color="7" fill="1" visible="yes" active="no"/>
+<layer number="22" name="bPlace" color="7" fill="1" visible="yes" active="no"/>
+<layer number="23" name="tOrigins" color="15" fill="1" visible="yes" active="no"/>
+<layer number="24" name="bOrigins" color="15" fill="1" visible="yes" active="no"/>
+<layer number="25" name="tNames" color="7" fill="1" visible="yes" active="no"/>
+<layer number="26" name="bNames" color="7" fill="1" visible="yes" active="no"/>
+<layer number="27" name="tValues" color="7" fill="1" visible="yes" active="no"/>
+<layer number="28" name="bValues" color="7" fill="1" visible="yes" active="no"/>
 <layer number="29" name="tStop" color="7" fill="3" visible="no" active="no"/>
 <layer number="30" name="bStop" color="7" fill="6" visible="no" active="no"/>
@@
 <layer number="35" name="tGlue" color="7" fill="4" visible="no" active="no"/>
 <layer number="36" name="bGlue" color="7" fill="5" visible="no" active="no"/>
-<layer number="37" name="tTest" color="7" fill="1" visible="no" active="no"/>
-<layer number="38" name="bTest" color="7" fill="1" visible="no" active="no"/>
+<layer number="37" name="tTest" color="7" fill="1" visible="yes" active="no"/>
+<layer number="38" name="bTest" color="7" fill="1" visible="yes" active="no"/>
 <layer number="39" name="tKeepout" color="4" fill="11" visible="no" active="no"/>
 <layer number="40" name="bKeepout" color="1" fill="11" visible="no" active="no"/>
@@
 <layer number="44" name="Drills" color="7" fill="1" visible="no" active="no"/>
 <layer number="45" name="Holes" color="7" fill="1" visible="no" active="no"/>
-<layer number="46" name="Milling" color="3" fill="1" visible="no" active="no"/>
-<layer number="47" name="Measures" color="7" fill="1" visible="no" active="no"/>
-<layer number="48" name="Document" color="7" fill="1" visible="no" active="no"/>
-<layer number="49" name="Reference" color="7" fill="1" visible="no" active="no"/>
-<layer number="50" name="dxf" color="7" fill="1" visible="no" active="no"/>
-<layer number="51" name="tDocu" color="7" fill="1" visible="no" active="no"/>
-<layer number="52" name="bDocu" color="7" fill="1" visible="no" active="no"/>
-<layer number="53" name="tGND_GNDA" color="7" fill="9" visible="no" active="no"/>
-<layer number="54" name="bGND_GNDA" color="1" fill="9" visible="no" active="no"/>
-<layer number="56" name="wert" color="7" fill="1" visible="no" active="no"/>
-<layer number="57" name="tCAD" color="7" fill="1" visible="no" active="no"/>
+<layer number="46" name="Milling" color="3" fill="1" visible="yes" active="no"/>
+<layer number="47" name="Measures" color="7" fill="1" visible="yes" active="no"/>
+<layer number="48" name="Document" color="7" fill="1" visible="yes" active="no"/>
+<layer number="49" name="Reference" color="7" fill="1" visible="yes" active="no"/>
+<layer number="50" name="dxf" color="7" fill="1" visible="yes" active="no"/>
+<layer number="51" name="tDocu" color="7" fill="1" visible="yes" active="no"/>
+<layer number="52" name="bDocu" color="7" fill="1" visible="yes" active="no"/>
+<layer number="53" name="tGND_GNDA" color="7" fill="9" visible="yes" active="no"/>
+<layer number="54" name="bGND_GNDA" color="1" fill="9" visible="yes" active="no"/>
+<layer number="56" name="wert" color="7" fill="1" visible="yes" active="no"/>
+<layer number="57" name="tCAD" color="7" fill="1" visible="yes" active="no"/>
 <layer number="90" name="Modules" color="5" fill="1" visible="yes" active="yes"/>
 <layer number="91" name="Nets" color="2" fill="1" visible="yes" active="yes"/>
@@
 </segment>
 <segment>
-<pinref part="IC$4" gate="G$1" pin="PB0"/>
-<wire x1="-25.4" y1="-43.18" x2="-25.4" y2="-45.72" width="0.1524" layer="91"/>
-<label x="-25.4" y="-45.72" size="1.778" layer="95" rot="R270" xref="yes"/>
-</segment>
-</net>
+<pinref part="IC$4" gate="G$1" pin="PB5"/>
+<wire x1="-30.48" y1="22.86" x2="-30.48" y2="25.4" width="0.1524" layer="91"/>
+<label x="-30.48" y="25.4" size="1.778" layer="95" rot="R90" xref="yes"/>
+</segment>
+</net>

Commit message: Some more (incomplete) work on ground plane connectivity.
Connections:
- net PIEZONEG: now also IC$4.PB0; no longer IC$4.PA10
Changed lines of the file:
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@@
-</segment>
-<segment>
-<pinref part="IC$4" gate="G$1" pin="PA10"/>
-<wire x1="0" y1="-12.7" x2="2.54" y2="-12.7" width="0.1524" layer="91"/>
-<label x="2.54" y="-12.7" size="1.778" layer="95" xref="yes"/>
 </segment>
 <segment>
@@
 <pinref part="ZN" gate="G$1" pin="P$1"/>
 </segment>
+<segment>
+<pinref part="IC$4" gate="G$1" pin="PB0"/>
+<wire x1="-25.4" y1="-43.18" x2="-25.4" y2="-45.72" width="0.1524" layer="91"/>
+<label x="-25.4" y="-45.72" size="1.778" layer="95" rot="R270" xref="yes"/>
+</segment>
 </net>

Commit message: More work on improving PCB layout.
Parts:
- removed R14: 10k, resistor:R-EU_R0402
Connections:
- removed net N$4: IC$1.EN, IC$1.VIN, J1.1
- new net N$8: C4.2, IC$1.EN, IC$1.VIN, J1.1
- net AVREG: no longer R14.2
- net INTEGCLR: no longer R14.1
- net VCC: no longer C4.2
- net VUSB: no longer R5.1
Changed lines of the file:
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@@
 <part name="C31" library="rcl" deviceset="C-EU" device="C0402" value="u1"/>
 <part name="R11" library="resistor" deviceset="R-EU_" device="R0402" value="500 (0.1%)"/>
-<part name="R14" library="resistor" deviceset="R-EU_" device="R0402" value="10k"/>
 <part name="R12" library="resistor" deviceset="R-EU_" device="R0402" value="500 (0.1%)"/>
 <part name="D6" library="adafruit" deviceset="DIODE" device="SOD-323F"/>
@@
 <instance part="GND26" gate="1" x="-148.844" y="-12.7" rot="R270"/>
 <instance part="IC$1" gate="G$1" x="-28.702" y="88.9"/>
-<instance part="P+3" gate="VCC" x="-63.5" y="93.98" rot="R90"/>
+<instance part="P+3" gate="VCC" x="-66.04" y="101.6" rot="R90"/>
 <instance part="C4" gate="G$1" x="-50.8" y="88.9" rot="R270"/>
 <instance part="C28" gate="G$1" x="-1.778" y="-118.618" rot="R90"/>
@@
 <instance part="C31" gate="G$1" x="177.8" y="-134.62" rot="R90"/>
 <instance part="R11" gate="G$1" x="71.12" y="-7.62" rot="R90"/>
-<instance part="R14" gate="G$1" x="55.88" y="-30.48" rot="R180"/>
 <instance part="R12" gate="G$1" x="109.22" y="-7.62" rot="R90"/>
 <instance part="D6" gate="G$1" x="-15.24" y="-86.36"/>
@@
 <segment>
 <pinref part="J1" gate="G$1" pin="2"/>
-<wire x1="-63.5" y1="101.6" x2="-60.96" y2="101.6" width="0.1524" layer="91"/>
-<wire x1="-63.5" y1="99.06" x2="-63.5" y2="101.6" width="0.1524" layer="91"/>
-<wire x1="-58.42" y1="99.06" x2="-63.5" y2="99.06" width="0.1524" layer="91"/>
 <pinref part="P+3" gate="VCC" pin="VCC"/>
-<wire x1="-58.42" y1="93.98" x2="-60.96" y2="93.98" width="0.1524" layer="91"/>
-<wire x1="-58.42" y1="93.98" x2="-58.42" y2="99.06" width="0.1524" layer="91"/>
-<junction x="-58.42" y="93.98"/>
-<pinref part="C4" gate="G$1" pin="2"/>
-<wire x1="-55.88" y1="88.9" x2="-58.42" y2="88.9" width="0.1524" layer="91"/>
-<wire x1="-58.42" y1="88.9" x2="-58.42" y2="93.98" width="0.1524" layer="91"/>
+<wire x1="-60.96" y1="101.6" x2="-63.5" y2="101.6" width="0.1524" layer="91"/>
 </segment>
 <segment>
@@
 <wire x1="-121.92" y1="-124.46" x2="-116.84" y2="-124.46" width="0.1524" layer="91"/>
 <pinref part="R16" gate="G$1" pin="1"/>
+</segment>
+<segment>
+<wire x1="-116.84" y1="60.96" x2="-119.38" y2="60.96" width="0.1524" layer="91"/>
+<label x="-119.38" y="60.96" size="1.778" layer="95" rot="R180" xref="yes"/>
 </segment>
 </net>
@@
 <wire x1="-132.08" y1="-38.1" x2="-137.16" y2="-38.1" width="0.1524" layer="91"/>
 <label x="-139.7" y="-48.26" size="1.778" layer="95" rot="R180" xref="yes"/>
-</segment>
-<segment>
-<pinref part="R5" gate="G$1" pin="1"/>
-<wire x1="-120.396" y1="60.96" x2="-116.078" y2="60.96" width="0.1524" layer="91"/>
-<label x="-119.38" y="60.96" size="1.778" layer="95" rot="R180" xref="yes"/>
 </segment>
 </net>
@@
 <wire x1="76.2" y1="-43.18" x2="76.2" y2="-38.1" width="0.1524" layer="91"/>
 <label x="76.2" y="-38.1" size="1.778" layer="95" rot="R90" xref="yes"/>
-</segment>
-<segment>
-<wire x1="58.42" y1="-20.32" x2="66.04" y2="-20.32" width="0.1524" layer="91"/>
-<wire x1="66.04" y1="-30.48" x2="66.04" y2="-20.32" width="0.1524" layer="91"/>
-<pinref part="R14" gate="G$1" pin="1"/>
-<wire x1="60.96" y1="-30.48" x2="66.04" y2="-30.48" width="0.1524" layer="91"/>
-<label x="58.42" y="-20.32" size="1.778" layer="95" rot="R180" xref="yes"/>
 </segment>
 <segment>
@@
 </segment>
 <segment>
-<pinref part="R14" gate="G$1" pin="2"/>
-<wire x1="50.8" y1="-30.48" x2="45.72" y2="-30.48" width="0.1524" layer="91"/>
-<label x="45.72" y="-30.48" size="1.778" layer="95" rot="R180" xref="yes"/>
-</segment>
-<segment>
 <pinref part="U$4" gate="G$1" pin="VCC"/>
 <wire x1="86.36" y1="-33.02" x2="91.44" y2="-33.02" width="0.1524" layer="91"/>
@@
 <pinref part="IC$10" gate="G$1" pin="IOUT"/>
 <wire x1="213.36" y1="-119.38" x2="218.44" y2="-119.38" width="0.1524" layer="91"/>
-</segment>
-</net>
-<net name="N$4" class="0">
-<segment>
-<wire x1="-41.402" y1="93.98" x2="-45.72" y2="93.98" width="0.1524" layer="91"/>
-<wire x1="-41.402" y1="83.82" x2="-45.72" y2="83.82" width="0.1524" layer="91"/>
-<wire x1="-45.72" y1="83.82" x2="-45.72" y2="93.98" width="0.1524" layer="91"/>
-<pinref part="IC$1" gate="G$1" pin="VIN"/>
-<pinref part="IC$1" gate="G$1" pin="EN"/>
-<pinref part="J1" gate="G$1" pin="1"/>
-<wire x1="-45.72" y1="93.98" x2="-45.72" y2="101.6" width="0.1524" layer="91"/>
-<junction x="-45.72" y="93.98"/>
 </segment>
 </net>
@@
 </segment>
 </net>
+<net name="N$8" class="0">
+<segment>
+<pinref part="C4" gate="G$1" pin="2"/>
+<wire x1="-55.88" y1="88.9" x2="-58.42" y2="88.9" width="0.1524" layer="91"/>
+<wire x1="-58.42" y1="88.9" x2="-58.42" y2="96.52" width="0.1524" layer="91"/>
+<wire x1="-41.402" y1="93.98" x2="-45.72" y2="93.98" width="0.1524" layer="91"/>
+<wire x1="-41.402" y1="83.82" x2="-45.72" y2="83.82" width="0.1524" layer="91"/>
+<wire x1="-45.72" y1="83.82" x2="-45.72" y2="93.98" width="0.1524" layer="91"/>
+<pinref part="IC$1" gate="G$1" pin="VIN"/>
+<pinref part="IC$1" gate="G$1" pin="EN"/>
+<pinref part="J1" gate="G$1" pin="1"/>
+<wire x1="-45.72" y1="93.98" x2="-45.72" y2="96.52" width="0.1524" layer="91"/>
+<junction x="-45.72" y="93.98"/>
+<wire x1="-45.72" y1="96.52" x2="-45.72" y2="101.6" width="0.1524" layer="91"/>
+<wire x1="-58.42" y1="96.52" x2="-45.72" y2="96.52" width="0.1524" layer="91"/>
+<junction x="-45.72" y="96.52"/>
+</segment>
+</net>

Commit message: Use recommended components for buck convertor and more work on layout
Parts:
- removed L1: 2u2, microbuilder:INDUCTOR_0603
- added I1: CDRH2D14, lightmeter:CDRH2D14
- C3, C4: device rcl:C-EUC0402 -> rcl:C-EUC0603
Connections:
- net N$10: now also I1.1; no longer L1.1
- net VREG: now also I1.2; no longer L1.2
Changed lines of the file:
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@@
 <part name="C10" library="rcl" deviceset="C-EU" device="C0402" value="4u7"/>
 <part name="GND3" library="supply1" deviceset="GND" device=""/>
-<part name="L1" library="microbuilder" deviceset="INDUCTOR" device="_0603" value="2u2"/>
 <part name="GND23" library="supply1" deviceset="GND" device=""/>
 <part name="P+1" library="supply1" deviceset="VCC" device=""/>
@@
 <part name="IC$1" library="lightmeter" deviceset="LM3671" device=""/>
 <part name="P+3" library="supply1" deviceset="VCC" device=""/>
-<part name="C4" library="rcl" deviceset="C-EU" device="C0402" value="4u7"/>
+<part name="C4" library="rcl" deviceset="C-EU" device="C0603" value="4u7"/>
 <part name="C28" library="rcl" deviceset="C-EU" device="C0402" value="4u7"/>
 <part name="GND28" library="supply1" deviceset="GND" device=""/>
@@
 <part name="U1" library="lightmeter" deviceset="USB-AB" device="USB-AB-MICRO-MIDMOUNT"/>
 <part name="GND24" library="supply1" deviceset="GND" device=""/>
-<part name="C3" library="rcl" deviceset="C-EU" device="C0402" value="10u"/>
+<part name="C3" library="rcl" deviceset="C-EU" device="C0603" value="10u"/>
 <part name="GND25" library="supply1" deviceset="GND" device=""/>
 <part name="U$6" library="lightmeter" deviceset="NLAS5223B" device=""/>
@@
 <part name="ZP" library="lightmeter" deviceset="WIREATTACHMENT" device=""/>
 <part name="ZN" library="lightmeter" deviceset="WIREATTACHMENT" device=""/>
+<part name="I1" library="lightmeter" deviceset="CDRH2D14" device=""/>
 </parts>
 <sheets>
@@
 <instance part="C10" gate="G$1" x="177.8" y="40.64" rot="R90"/>
 <instance part="GND3" gate="1" x="195.58" y="-20.32" rot="R270"/>
-<instance part="L1" gate="G$1" x="-10.16" y="93.98"/>
 <instance part="GND23" gate="1" x="-48.26" y="73.66"/>
 <instance part="P+1" gate="VCC" x="-114.3" y="-33.02" rot="R270"/>
@@
 <instance part="ZP" gate="G$1" x="108.712" y="59.182"/>
 <instance part="ZN" gate="G$1" x="108.712" y="49.022"/>
+<instance part="I1" gate="G$1" x="-10.16" y="93.98"/>
 </instances>
 <busses>
@@
 </segment>
 <segment>
-<pinref part="L1" gate="G$1" pin="2"/>
-<wire x1="-5.08" y1="93.98" x2="2.54" y2="93.98" width="0.1524" layer="91"/>
-<wire x1="-5.08" y1="93.98" x2="-5.08" y2="106.68" width="0.1524" layer="91"/>
-<junction x="-5.08" y="93.98"/>
-<wire x1="-5.08" y1="106.68" x2="7.62" y2="106.68" width="0.1524" layer="91"/>
-<label x="7.62" y="106.68" size="1.778" layer="95" xref="yes"/>
+<wire x1="-5.08" y1="93.98" x2="-2.54" y2="93.98" width="0.1524" layer="91"/>
 <pinref part="IC$1" gate="G$1" pin="FB"/>
+<wire x1="-2.54" y1="93.98" x2="2.54" y2="93.98" width="0.1524" layer="91"/>
 <wire x1="-16.002" y1="88.9" x2="2.54" y2="88.9" width="0.1524" layer="91"/>
 <wire x1="2.54" y1="88.9" x2="2.54" y2="93.98" width="0.1524" layer="91"/>
@@
 <junction x="2.54" y="93.98"/>
 <pinref part="C3" gate="G$1" pin="1"/>
+<pinref part="I1" gate="G$1" pin="2"/>
+<wire x1="-2.54" y1="106.68" x2="7.62" y2="106.68" width="0.1524" layer="91"/>
+<label x="7.62" y="106.68" size="1.778" layer="95" xref="yes"/>
+<wire x1="-2.54" y1="106.68" x2="-2.54" y2="93.98" width="0.1524" layer="91"/>
+<junction x="-2.54" y="93.98"/>
 </segment>
 <segment>
@@
 <segment>
 <pinref part="IC$1" gate="G$1" pin="SW"/>
-<pinref part="L1" gate="G$1" pin="1"/>
 <wire x1="-16.002" y1="93.98" x2="-15.24" y2="93.98" width="0.1524" layer="91"/>
-</segment>
-</net>
+<pinref part="I1" gate="G$1" pin="1"/>
+</segment>
+</net>
